Commit message: Rebuild timda_mobile_platform.urdf by Solidworks

File: timda_description/urdf/timda_mobile_platform.urdf (robot description, URDF)
Before this commit: robot timda_mobile_platform, 1 links, 0 joints
Links:
- link base_link: mass 45 -> 50

File: timda_description/urdf/timda_mobile_platform.urdf.xacro (robot description, xacro)
@@ -7,5 +7,5 @@
   <link name="base_footprint"/>
   <joint name="base_link_joint" type="fixed">
-    <origin xyz="0.0 0 0.01" rpy="0 0 0" />
+    <origin xyz="0.0 0 0.0" rpy="0 0 0" />
     <parent link="base_footprint"/>
     <child link="base_link" />
@@ -14,14 +14,15 @@
     <inertial>
       <origin
-        xyz="-0.074645 -4.8E-06 0.12685"
+        xyz="-0.075595 -4.8123E-06 0.13958"
         rpy="0 0 0" />
-      <mass value="45" />
+      <mass
+        value="50" />
       <inertia
-        ixx="0.13639"
-        ixy="-0.00052166"
-        ixz="-4.6978E-05"
-        iyy="0.11714"
-        iyz="3.4276E-05"
-        izz="0.22097" />
+        ixx="0.13635"
+        ixy="-0.00051122"
+        ixz="-6.0686E-05"
+        iyy="0.11712"
+        iyz="2.0569E-05"
+        izz="0.22093" />
     </inertial>
     <visual>

Commit message: Rebuild robot's urdf with setting materials

File: timda_description/urdf/timda_mobile_platform.urdf (robot description, URDF)
Before this commit: robot timda_mobile_platform, 1 links, 0 joints
Links:
- link base_link: mass 50 -> 31.314; geometry collision mesh filename=package://timda_mobile/meshes/base_link.STL; visual mesh filename=package://timda_mobile/meshes/base_link.STL

File: timda_description/urdf/timda_mobile_platform.urdf.xacro (robot description, xacro)
@@ -27,15 +27,15 @@
     <inertial>
       <origin
-        xyz="-0.075595 -4.8123E-06 0.13958"
+        xyz="-0.03475 -0.00014056 0.15811"
         rpy="0 0 0" />
       <mass
-        value="50" />
+        value="31.314" />
       <inertia
-        ixx="0.13635"
-        ixy="-0.00051122"
-        ixz="-6.0686E-05"
-        iyy="0.11712"
-        iyz="2.0569E-05"
-        izz="0.22093" />
+        ixx="0.29031"
+        ixy="-0.0013778"
+        ixz="-0.00016386"
+        iyy="0.25069"
+        iyz="5.56E-05"
+        izz="0.48464" />
     </inertial>
     <visual>
