Commit message: Add 2 hokuyo utm30lx lidar to timda mobile in Gazebo

File: timda_description/urdf/timda_mobile_platform.urdf.xacro (robot description, xacro)
@@ -4,5 +4,18 @@
      For more information, please see http://wiki.ros.org/sw_urdf_exporter -->
 <robot xmlns:xacro="http://www.ros.org/wiki/xacro" name="timda_mobile_platform">
+  <xacro:property name="M_PI" value="3.14159265359" />
+  <xacro:property name="M_PI_2" value="1.57079632679" />
   <xacro:include filename="$(find timda_description)/urdf/timda_mobile_platform.gazebo.xacro" />
+  <xacro:include filename="$(find hector_sensors_description)/urdf/hokuyo_utm30lx.urdf.xacro" />
+  <xacro:hokuyo_utm30lx name="front" parent="base_link" ros_topic="laser_front"
+                        update_rate="30" ray_count="270"
+                        min_angle="-135" max_angle="135">
+    <origin xyz="0.38516904756 0.28066904756 0.11" rpy="${M_PI} 0 ${M_PI/4}" />
+  </xacro:hokuyo_utm30lx>
+  <xacro:hokuyo_utm30lx name="back" parent="base_link" ros_topic="laser_back"
+                        update_rate="30" ray_count="270"
+                        min_angle="-135" max_angle="135">
+    <origin xyz="-0.38616904756 -0.28066904756 0.11" rpy="${M_PI} 0 ${M_PI/4+M_PI}" />
+  </xacro:hokuyo_utm30lx>
   <link name="base_footprint"/>
   <joint name="base_link_joint" type="fixed">

Commit message: Modify footprint and let weight to be 0
Let weight be 0 is because planar move plugin

File: timda_description/urdf/timda_mobile_platform.urdf.xacro (robot description, xacro)
@@ -18,7 +18,14 @@
     <origin xyz="-0.38616904756 -0.28066904756 0.11" rpy="${M_PI} 0 ${M_PI/4+M_PI}" />
   </xacro:hokuyo_utm30lx>
-  <link name="base_footprint"/>
+  <link name="base_footprint">
+    <visual>
+      <origin xyz="0 0 0" rpy="0 0 0" />
+      <geometry>
+        <box size="0.001 0.001 0.001" />
+      </geometry>
+    </visual>
+  </link>
   <joint name="base_link_joint" type="fixed">
-    <origin xyz="0.0 0 0.0" rpy="0 0 0" />
+    <origin xyz="0.0 0 0.05" rpy="0 0 0" />
     <parent link="base_footprint"/>
     <child link="base_link" />
@@ -30,5 +37,5 @@
         rpy="0 0 0" />
       <mass
-        value="31.314" />
+        value="0.0" />
       <inertia
         ixx="0.29031"
