Commit message: Remove suction vaccum gripper

File: mobile_description/urdf/timda_mobile_platform.gazebo.xacro (robot description, xacro)
@@ -15,4 +15,6 @@
     </gazebo>
     <gazebo reference="${prefix}base_link">
+      <mu1>0.0</mu1>
+      <mu2>0.0</mu2>
       <material>Gazebo/DarkGrey</material>
     </gazebo>

File: mobile_description/urdf/timda_mobile_platform.urdf.xacro (robot description, xacro)
@@ -54,4 +54,12 @@
             filename="package://mobile_description/meshes/base_link.STL" />
         </geometry>
+        <surface>
+          <friction>
+            <ode>
+              <mu>0.0</mu>
+              <mu2>0.0</mu2>
+            </ode>
+          </friction>
+        </surface>
       </collision>
     </link>

File: mobile_description/urdf/timda_mobile_platform_sim_odom.urdf.xacro (robot description, xacro)
@@ -23,5 +23,5 @@
         <origin xyz="0 0 0" rpy="0 0 0" />
         <geometry>
-          <box size="0.001 0.001 0.001" />
+          <box size="0.01 0.01 0.01" />
         </geometry>
       </visual>
@@ -68,4 +68,12 @@
             filename="package://mobile_description/meshes/base_link.STL" />
         </geometry>
+        <surface>
+          <friction>
+            <ode>
+              <mu>0.0</mu>
+              <mu2>0.0</mu2>
+            </ode>
+          </friction>
+        </surface>
       </collision>
     </link>

File: single_arm_description/urdf/single_arm.gazebo.xacro (robot description, xacro)
@@ -71,7 +71,4 @@
   </gazebo>
   <gazebo reference="${side}_joint_6">
-    <implicitSpringDamper>True</implicitSpringDamper>
-  </gazebo>
-  <gazebo reference="${side}_joint_7">
     <implicitSpringDamper>True</implicitSpringDamper>
   </gazebo>

File: single_arm_description/urdf/single_arm.transmission.xacro (robot description, xacro)
@@ -62,4 +62,5 @@
     </actuator>
   </transmission>
+<!--
   <transmission name="${side}_tran7">
     <type>transmission_interface/SimpleTransmission</type>
@@ -71,5 +72,5 @@
       <mechanicalReduction>1</mechanicalReduction>
     </actuator>
-  </transmission>
+  </transmission> -->
 </xacro:macro>
 </robot>

File: single_arm_description/urdf/single_arm.xacro (robot description, xacro)
@@ -5,5 +5,5 @@
   <xacro:include filename="$(find single_arm_description)/urdf/materials.xacro" />
   <!-- Constants for robot dimensions -->
-  <xacro:macro name="single_arm" params="side parent child toolrot *origin">
+  <xacro:macro name="single_arm" params="side parent *origin">
 	  <link
 	    name="${side}_Base">
@@ -417,5 +417,5 @@
 	    </collision>
 	  </link> -->
-		<joint
+		<!-- <joint
 			name="${side}_joint_7"
 			type="revolute">
@@ -423,7 +423,4 @@
 				xyz="0 0.03680 0.135"
 				rpy="0 0 ${toolrot}" />
-				<!-- rpy="1.5708 ${toolrot} 0" /> -->
-				<!-- xyz="-0.008041 0.038 0.13545" -->
-				<!-- xyz="-0.0025 0.038 0.135" -->
 			<parent
 				link="${side}_Link_6" />
@@ -438,5 +435,5 @@
                 velocity="6.5" />
           <dynamics damping="0.7"/>
-		</joint>
+		</joint> -->
           <!--
 	  <link

File: timda_description/urdf/timda.gazebo.xacro (robot description, xacro)
@@ -14,299 +14,3 @@
     </plugin>
   </gazebo>
-  <gazebo>
-    <plugin name="gazebo_ros_vacuum_gripper" filename="libgazebo_ros_vacuum_gripper.so">
-      <robotNamespace>/robot/left_gazebo/vacuum_gripper1</robotNamespace>
-      <bodyName>l_end_Link1</bodyName>
-      <topicName>grasping</topicName>
-      <maxForce>50</maxForce>
-      <maxDistance>0.05</maxDistance>
-      <minDistance>0.01</minDistance>
-    </plugin>
-  </gazebo>
-  <gazebo>
-    <plugin name="gazebo_ros_vacuum_gripper" filename="libgazebo_ros_vacuum_gripper.so">
-      <robotNamespace>/robot/left_gazebo/vacuum_gripper2</robotNamespace>
-      <bodyName>l_end_Link2</bodyName>
-      <topicName>grasping</topicName>
-      <maxForce>50</maxForce>
-      <maxDistance>0.05</maxDistance>
-      <minDistance>0.01</minDistance>
-    </plugin>
-  </gazebo>
-  <gazebo>
-    <plugin name="gazebo_ros_vacuum_gripper" filename="libgazebo_ros_vacuum_gripper.so">
-      <robotNamespace>/robot/left_gazebo/vacuum_gripper3</robotNamespace>
-      <bodyName>l_end_Link3</bodyName>
-      <topicName>grasping</topicName>
-      <maxForce>50</maxForce>
-      <maxDistance>0.05</maxDistance>
-      <minDistance>0.01</minDistance>
-    </plugin>
-  </gazebo>
-  <gazebo>
-    <plugin name="gazebo_ros_vacuum_gripper" filename="libgazebo_ros_vacuum_gripper.so">
-      <robotNamespace>/robot/left_gazebo/vacuum_gripper4</robotNamespace>
-      <bodyName>l_end_Link4</bodyName>
-      <topicName>grasping</topicName>
-      <maxForce>50</maxForce>
-      <maxDistance>0.05</maxDistance>
-      <minDistance>0.01</minDistance>
-    </plugin>
-  </gazebo>
-  <gazebo>
-    <plugin name="gazebo_ros_vacuum_gripper" filename="libgazebo_ros_vacuum_gripper.so">
-      <robotNamespace>/robot/left_gazebo/vacuum_gripper5</robotNamespace>
-      <bodyName>l_end_Link5</bodyName>
-      <topicName>grasping</topicName>
-      <maxForce>50</maxForce>
-      <maxDistance>0.05</maxDistance>
-      <minDistance>0.01</minDistance>
-    </plugin>
-  </gazebo>
-  <gazebo>
-    <plugin name="gazebo_ros_vacuum_gripper" filename="libgazebo_ros_vacuum_gripper.so">
-      <robotNamespace>/robot/right_gazebo/vacuum_gripper1</robotNamespace>
-      <bodyName>r_end_Link1</bodyName>
-      <topicName>grasping</topicName>
-      <maxForce>50</maxForce>
-      <maxDistance>0.05</maxDistance>
-      <minDistance>0.01</minDistance>
-    </plugin>
-  </gazebo>
-  <gazebo>
-    <plugin name="gazebo_ros_vacuum_gripper" filename="libgazebo_ros_vacuum_gripper.so">
-      <robotNamespace>/robot/right_gazebo/vacuum_gripper2</robotNamespace>
-      <bodyName>r_end_Link2</bodyName>
-      <topicName>grasping</topicName>
-      <maxForce>50</maxForce>
-      <maxDistance>0.05</maxDistance>
-      <minDistance>0.01</minDistance>
-    </plugin>
-  </gazebo>
-  <gazebo>
-    <plugin name="gazebo_ros_vacuum_gripper" filename="libgazebo_ros_vacuum_gripper.so">
-      <robotNamespace>/robot/right_gazebo/vacuum_gripper3</robotNamespace>
-      <bodyName>r_end_Link3</bodyName>
-      <topicName>grasping</topicName>
-      <maxForce>50</maxForce>
-      <maxDistance>0.05</maxDistance>
-      <minDistance>0.01</minDistance>
-    </plugin>
-  </gazebo>
-  <gazebo>
-    <plugin name="gazebo_ros_vacuum_gripper" filename="libgazebo_ros_vacuum_gripper.so">
-      <robotNamespace>/robot/right_gazebo/vacuum_gripper4</robotNamespace>
-      <bodyName>r_end_Link4</bodyName>
-      <topicName>grasping</topicName>
-      <maxForce>50</maxForce>
-      <maxDistance>0.05</maxDistance>
-      <minDistance>0.01</minDistance>
-    </plugin>
-  </gazebo>
-  <gazebo>
-    <plugin name="gazebo_ros_vacuum_gripper" filename="libgazebo_ros_vacuum_gripper.so">
-      <robotNamespace>/robot/right_gazebo/vacuum_gripper5</robotNamespace>
-      <bodyName>r_end_Link5</bodyName>
-      <topicName>grasping</topicName>
-      <maxForce>50</maxForce>
-      <maxDistance>0.05</maxDistance>
-      <minDistance>0.01</minDistance>
-    </plugin>
-  </gazebo>
-  <gazebo reference="Bin">
-    <mu1>200</mu1>
-    <mu2>200</mu2>
-    <material>Gazebo/Blue</material>
-    <selfCollide>false</selfCollide>
-  </gazebo>
-<!--====================================================================================
-<gazebo reference="Base">
-    <mu1>0.5</mu1>
-    <mu2>0.5</mu2>
-    <material>Gazebo/Orange</material>
-    <selfCollide>false</selfCollide>
-  </gazebo>
-  <gazebo reference="Link_1">
-    <mu1>0.5</mu1>
-    <mu2>0.5</mu2>
-    <material>Gazebo/Black</material>
-    <selfCollide>false</selfCollide>
-  </gazebo>
-  <gazebo reference="Link_2">
-    <mu1>0.5</mu1>
-    <mu2>0.5</mu2>
-    <material>Gazebo/Orange</material>
-    <selfCollide>false</selfCollide>
-  </gazebo>
-  <gazebo reference="Link_3">
-    <mu1>0.5</mu1>
-    <mu2>0.5</mu2>
-    <material>Gazebo/Black</material>
-    <selfCollide>false</selfCollide>
-  </gazebo>
-  <gazebo reference="Link_4">
-    <mu1>0.5</mu1>
-    <mu2>0.5</mu2>
-    <material>Gazebo/Orange</material>
-    <selfCollide>false</selfCollide>
-  </gazebo>
-  <gazebo reference="Link_5">
-    <mu1>0.5</mu1>
-    <mu2>0.5</mu2>
-    <material>Gazebo/Black</material>
-    <selfCollide>false</selfCollide>
-  </gazebo>
-  <gazebo reference="Link_6">
-    <mu1>0.5</mu1>
-    <mu2>0.5</mu2>
-    <material>Gazebo/Orange</material>
-    <selfCollide>false</selfCollide>
-  </gazebo>
-  <gazebo reference="Arm_Base_R">
-    <mu1>0.5</mu1>
-    <mu2>0.5</mu2>
-    <material>Gazebo/Orange</material>
-    <selfCollide>false</selfCollide>
-  </gazebo>
-  <gazebo reference="Link_R_1">
-    <mu1>0.5</mu1>
-    <mu2>0.5</mu2>
-    <material>Gazebo/Black</material>
-    <selfCollide>false</selfCollide>
-  </gazebo>
-  <gazebo reference="Link_R_2">
-    <mu1>0.5</mu1>
-    <mu2>0.5</mu2>
-    <material>Gazebo/Orange</material>
-    <selfCollide>false</selfCollide>
-  </gazebo>
-  <gazebo reference="Link_R_3">
-    <mu1>0.5</mu1>
-    <mu2>0.5</mu2>
-    <material>Gazebo/Black</material>
-    <selfCollide>false</selfCollide>
-  </gazebo>
-  <gazebo reference="Link_R_4">
-    <mu1>0.5</mu1>
-    <mu2>0.5</mu2>
-    <material>Gazebo/Orange</material>
-    <selfCollide>false</selfCollide>
-  </gazebo>
-  <gazebo reference="Link_R_5">
-    <mu1>0.5</mu1>
-    <mu2>0.5</mu2>
-    <material>Gazebo/Black</material>
-    <selfCollide>false</selfCollide>
-  </gazebo>
-  <gazebo reference="Link_R_6">
-    <mu1>0.5</mu1>
-    <mu2>0.5</mu2>
-    <material>Gazebo/Orange</material>
-    <selfCollide>false</selfCollide>
-  </gazebo>
-================================================================-->
-<!--
-  <gazebo reference="Link_7">
-    <mu1>0.2</mu1>
-    <mu2>0.2</mu2>
-    <material>Gazebo/Black</material>
-    <selfCollide>true</selfCollide>
-  </gazebo>
-  <gazebo reference="Link_8">
-    <mu1>0.2</mu1>
-    <mu2>0.2</mu2>
-    <material>Gazebo/Orange</material>
-    <selfCollide>false</selfCollide>
-  </gazebo>
--->
-  <!-- camera_link -->
-  <!--gazebo reference="camera_link">
-    <mu1>0.2</mu1>
-    <mu2>0.2</mu2>
-    <material>Gazebo/Red</material>
-    <selfCollide>false</selfCollide>
-  </gazebo-->
-  <!-- hokuyo -->
-  <!--gazebo reference="hokuyo_link">
-    <sensor type="gpu_ray" name="head_hokuyo_sensor">
-      <pose>0 0 0 0 0 0</pose>
-      <visualize>false</visualize>
-      <update_rate>40</update_rate>
-      <ray>
-        <scan>
-          <horizontal>
-            <samples>720</samples>
-            <resolution>1</resolution>
-            <min_angle>-1.570796</min_angle>
-            <max_angle>1.570796</max_angle>
-          </horizontal>
-        </scan>
-        <range>
-          <min>0.10</min>
-          <max>30.0</max>
-          <resolution>0.01</resolution>
-        </range>
-        <noise>
-          <type>gaussian</type>
-          <!- Noise parameters based on published spec for Hokuyo laser
-               achieving "+-30mm" accuracy at range < 10m.  A mean of 0.0m and
-               stddev of 0.01m will put 99.7% of samples within 0.03m of the true
-               reading. ->
-          <mean>0.0</mean>
-          <stddev>0.01</stddev>
-        </noise>
-      </ray>
-      <plugin name="gazebo_ros_head_hokuyo_controller" filename="libgazebo_ros_gpu_laser.so">
-        <topicName>/rrbot/laser/scan</topicName>
-        <frameName>hokuyo_link</frameName>
-      </plugin>
-    </sensor>
-  </gazebo-->
-  <!-- camera -->
-  <!--gazebo reference="camera_link">
-    <sensor type="camera" name="camera1">
-      <update_rate>30.0</update_rate>
-      <camera name="head">
-        <horizontal_fov>1.3962634</horizontal_fov>
-        <image>
-          <width>800</width>
-          <height>800</height>
-          <format>R8G8B8</format>
-        </image>
-        <clip>
-          <near>0.02</near>
-          <far>300</far>
-        </clip>
-        <noise>
-          <type>gaussian</type>
-          <!- Noise is sampled independently per pixel on each frame.
-               That pixel's noise value is added to each of its color
-               channels, which at that point lie in the range [0,1]. ->
-          <mean>0.0</mean>
-          <stddev>0.007</stddev>
-        </noise>
-      </camera>
-      <plugin name="camera_controller" filename="libgazebo_ros_camera.so">
-        <alwaysOn>true</alwaysOn>
-        <updateRate>0.0</updateRate>
-        <cameraName>urdf_0129/camera1</cameraName>
-        <imageTopicName>image_raw</imageTopicName>
-        <cameraInfoTopicName>camera_info</cameraInfoTopicName>
-        <frameName>camera_link_optical</frameName>
-        <!- setting hackBaseline to anything but 0.0 will cause a misalignment
-            between the gazebo sensor image and the frame it is supposed to
-            be attached to ->
-        <hackBaseline>0.0</hackBaseline>
-        <distortionK1>0.0</distortionK1>
-        <distortionK2>0.0</distortionK2>
-        <distortionK3>0.0</distortionK3>
-        <distortionT1>0.0</distortionT1>
-        <distortionT2>0.0</distortionT2>
-        <CxPrime>0</CxPrime>
-        <Cx>0.0</Cx>
-        <Cy>0.0</Cy>
-        <focalLength>0.0</focalLength>
-      </plugin>
-    </sensor>
-  </gazebo-->
 </robot>

File: timda_description/urdf/timda.urdf.xacro (robot description, xacro)
@@ -5,5 +5,5 @@
   <xacro:include filename="$(find timda_body_description)/urdf/timda_body.xacro" />
   <!-- <xacro:include filename="$(find slide_rail)/urdf/slide_rail.xacro" /> -->
-  <xacro:include filename="$(find suction_description)/urdf/suction_urdf.xacro" />
+  <!-- <xacro:include filename="$(find suction_description)/urdf/suction_urdf.xacro" /> -->
   <!--xacro:include filename="$(find single_arm_description)/urdf/materials.xacro" /-->
   <xacro:include filename="$(find timda_description)/urdf/timda.gazebo.xacro" />
@@ -13,23 +13,19 @@
       xyz="0.047646 0.0 0.3"
       rpy="0 0 0" />
-    <!--0.037646-->
-    <!--<origin
-      xyz="0 0 0.562"
-      rpy="0 0 0" /-->
     <parent link="mobile_base_link"/>
     <child link="base_link"/>
   </joint>
   <xacro:timda_mobile_platform prefix="mobile_"/>
-  <xacro:single_arm side="r"  parent="slide_right" child="r_tool_link" toolrot="-1.57">
+  <xacro:single_arm side="r"  parent="slide_right">
     <origin xyz="0.0 0.1151 0.0" rpy="1.57 3.1415926 3.1415926" />
   </xacro:single_arm>
-  <xacro:suction side="r"  parent="r_Link_6">
+  <!-- <xacro:suction side="r"  parent="r_Link_6">
     <origin xyz="0 -0.016 0" rpy="0 0 -1.57" />
-  </xacro:suction>
-  <xacro:single_arm side="l"  parent="slide_left" child="l_tool_link" toolrot="1.57">
+  </xacro:suction> -->
+  <xacro:single_arm side="l"  parent="slide_left">
     <origin xyz="0.0 0.1151 0.0" rpy="-1.57 0 0" />
   </xacro:single_arm>
-  <xacro:suction side="l"  parent="l_Link_6">
+  <!-- <xacro:suction side="l"  parent="l_Link_6">
     <origin xyz="0 0.016 0" rpy="0 0 1.57" />
-  </xacro:suction>
+  </xacro:suction> -->
 </robot>

File: timda_description/urdf/timda_sim_odom.urdf.xacro (robot description, xacro)
@@ -13,23 +13,19 @@
       xyz="0.047646 0.0 0.3"
       rpy="0 0 0" />
-    <!--0.037646-->
-    <!--<origin
-      xyz="0 0 0.562"
-      rpy="0 0 0" /-->
     <parent link="mobile_base_link"/>
     <child link="base_link"/>
   </joint>
   <xacro:timda_mobile_platform prefix="mobile_"/>
-  <xacro:single_arm side="r"  parent="slide_right" child="r_tool_link" toolrot="-1.57">
+  <xacro:single_arm side="r"  parent="slide_right">
     <origin xyz="0.0 0.1151 0.0" rpy="1.57 3.1415926 3.1415926" />
   </xacro:single_arm>
-  <xacro:suction side="r"  parent="r_Link_6">
+  <!-- <xacro:suction side="r"  parent="r_Link_6">
     <origin xyz="0 -0.016 0" rpy="0 0 -1.57" />
-  </xacro:suction>
-  <xacro:single_arm side="l"  parent="slide_left" child="l_tool_link" toolrot="1.57">
+  </xacro:suction> -->
+  <xacro:single_arm side="l"  parent="slide_left">
     <origin xyz="0.0 0.1151 0.0" rpy="-1.57 0 0" />
   </xacro:single_arm>
-  <xacro:suction side="l"  parent="l_Link_6">
+  <!-- <xacro:suction side="l"  parent="l_Link_6">
     <origin xyz="0 0.016 0" rpy="0 0 1.57" />
-  </xacro:suction>
+  </xacro:suction> -->
 </robot>
