Commit message: Hot fix

File: mobile_description/urdf/timda_mobile_platform.urdf.xacro (robot description, xacro)
@@ -6,4 +6,5 @@
   <xacro:property name="M_PI" value="3.14159265359" />
   <xacro:property name="M_PI_2" value="1.57079632679" />
+  <xacro:include filename="$(find mobile_description)/urdf/timda_mobile_platform.gazebo.xacro" />
   <xacro:include filename="$(find hector_sensors_description)/urdf/hokuyo_utm30lx.urdf.xacro" />
   <xacro:macro name="timda_mobile_platform" params="prefix">

File: timda_body_description/urdf/timda_body.gazebo.xacro (robot description, xacro)
@@ -1,27 +1,29 @@
 <?xml version="1.0"?>
 <robot xmlns:xacro="http://www.ros.org/wiki/xacro">
-  <gazebo reference="base_link">
-    <mu1>0.2</mu1>
-    <mu2>0.2</mu2>
-    <material>Gazebo/Gray</material>
-    <selfCollide>false</selfCollide>
-  </gazebo>
-  <gazebo reference="slide_right">
-    <mu1>0.2</mu1>
-    <mu2>0.2</mu2>
-    <material>Gazebo/Black</material>
-    <selfCollide>false</selfCollide>
-  </gazebo>
-  <gazebo reference="slide_left">
-    <mu1>0.2</mu1>
-    <mu2>0.2</mu2>
-    <material>Gazebo/Black</material>
-    <selfCollide>false</selfCollide>
-  </gazebo>
-  <gazebo reference="joint_right">
-    <implicitSpringDamper>True</implicitSpringDamper>
-  </gazebo>
-  <gazebo reference="joint_left">
-    <implicitSpringDamper>True</implicitSpringDamper>
-  </gazebo>
+  <xacro:macro name="timda_body_gazebo" params="prefix">
+    <gazebo reference="${prefix}base_link">
+      <mu1>0.2</mu1>
+      <mu2>0.2</mu2>
+      <material>Gazebo/Gray</material>
+      <selfCollide>false</selfCollide>
+    </gazebo>
+    <gazebo reference="${prefix}slide_right">
+      <mu1>0.2</mu1>
+      <mu2>0.2</mu2>
+      <material>Gazebo/Black</material>
+      <selfCollide>false</selfCollide>
+    </gazebo>
+    <gazebo reference="${prefix}slide_left">
+      <mu1>0.2</mu1>
+      <mu2>0.2</mu2>
+      <material>Gazebo/Black</material>
+      <selfCollide>false</selfCollide>
+    </gazebo>
+    <gazebo reference="${prefix}joint_right">
+      <implicitSpringDamper>True</implicitSpringDamper>
+    </gazebo>
+    <gazebo reference="${prefix}joint_left">
+      <implicitSpringDamper>True</implicitSpringDamper>
+    </gazebo>
+  </xacro:macro>
 </robot>

File: timda_body_description/urdf/timda_body.xacro (robot description, xacro)
@@ -4,181 +4,184 @@
   xmlns:xacro="http://www.ros.org/wiki/xacro">
   <xacro:include filename="$(find timda_body_description)/urdf/timda_body.gazebo.xacro" />
-  <link
-    name="base_link">
-    <inertial>
+  <xacro:macro name="timda_body" params="prefix">
+    <link
+      name="${prefix}base_link">
+      <inertial>
+        <origin
+          xyz="0.0 0 0"
+          rpy="0 0 0" />
+        <mass
+          value="2.072" />
+        <inertia
+          ixx="1"
+          ixy="0"
+          ixz="0"
+          iyy="1"
+          iyz="0"
+          izz="1" />
+      </inertial>
+      <visual>
+        <origin
+          xyz="0 0 0"
+          rpy="0 0 0" />
+        <geometry>
+          <mesh
+            filename="package://timda_body_description/meshes/base_link.STL" />
+        </geometry>
+        <material
+          name="">
+          <color
+            rgba="0.79216 0.81961 0.93333 1" />
+        </material>
+      </visual>
+      <collision>
+        <origin
+          xyz="0 0 0"
+          rpy="0 0 0" />
+        <geometry>
+          <mesh
+            filename="package://timda_body_description/meshes/base_link.STL" />
+        </geometry>
+      </collision>
+    </link>
+    <link
+      name="${prefix}slide_right">
+      <inertial>
+        <origin
+          xyz="1.5718E-05 -0.006626 2.4586E-06"
+          rpy="0 0 0" />
+        <mass
+          value="0.24709" />
+        <inertia
+          ixx="1"
+          ixy="0"
+          ixz="0"
+          iyy="1"
+          iyz="0"
+          izz="1" />
+      </inertial>
+      <visual>
+        <origin
+          xyz="0 0 0"
+          rpy="0 0 0" />
+        <geometry>
+          <mesh
+            filename="package://timda_body_description/meshes/slide_right.STL" />
+        </geometry>
+        <material
+          name="">
+          <color
+            rgba="0.89804 0.91765 0.92941 1" />
+        </material>
+      </visual>
+      <collision>
+        <origin
+          xyz="0 0 0"
+          rpy="0 0 0" />
+        <geometry>
+          <mesh
+            filename="package://timda_body_description/meshes/slide_right.STL" />
+        </geometry>
+      </collision>
+    </link>
+    <joint
+      name="${prefix}joint_right"
+      type="prismatic">
       <origin
-        xyz="0.0 0 0"
+        xyz="-0.2 0.0765 1.1815"
         rpy="0 0 0" />
-      <mass
-        value="2.072" />
-      <inertia
-        ixx="1"
-        ixy="0"
-        ixz="0"
-        iyy="1"
-        iyz="0"
-        izz="1" />
-    </inertial>
-    <visual>
+      <parent
+        link="${prefix}base_link" />
+      <child
+        link="${prefix}slide_right" />
+      <axis
+        xyz="0 0 1" />
+      <limit
+        lower="-0.8"
+        upper="0"
+        effort="9000"
+        velocity="6.5" />
+      <dynamics damping="7"/>
+    </joint>
+    <link
+      name="${prefix}slide_left">
+      <inertial>
+        <origin
+          xyz="-1.5722E-05 0.006626 2.4586E-06"
+          rpy="0 0 0" />
+        <mass
+          value="0.24709" />
+        <inertia
+          ixx="1"
+          ixy="0"
+          ixz="0"
+          iyy="1"
+          iyz="0"
+          izz="1" />
+      </inertial>
+      <visual>
+        <origin
+          xyz="0 0 0"
+          rpy="0 0 0" />
+        <geometry>
+          <mesh
+            filename="package://timda_body_description/meshes/slide_right.STL" />
+        </geometry>
+        <material
+          name="">
+          <color
+            rgba="0.89804 0.91765 0.92941 1" />
+        </material>
+      </visual>
+      <collision>
+        <origin
+          xyz="0 0 0"
+          rpy="0 0 0" />
+        <geometry>
+          <mesh
+            filename="package://timda_body_description/meshes/slide_right.STL" />
+        </geometry>
+      </collision>
+    </link>
+    <joint
+      name="${prefix}joint_left"
+      type="prismatic">
       <origin
-        xyz="0 0 0"
-        rpy="0 0 0" />
-      <geometry>
-        <mesh
-          filename="package://timda_body_description/meshes/base_link.STL" />
-      </geometry>
-      <material
-        name="">
-        <color
-          rgba="0.79216 0.81961 0.93333 1" />
-      </material>
-    </visual>
-    <collision>
-      <origin
-        xyz="0 0 0"
-        rpy="0 0 0" />
-      <geometry>
-        <mesh
-          filename="package://timda_body_description/meshes/base_link.STL" />
-      </geometry>
-    </collision>
-  </link>
-  <link
-    name="slide_right">
-    <inertial>
-      <origin
-        xyz="1.5718E-05 -0.006626 2.4586E-06"
-        rpy="0 0 0" />
-      <mass
-        value="0.24709" />
-      <inertia
-        ixx="1"
-        ixy="0"
-        ixz="0"
-        iyy="1"
-        iyz="0"
-        izz="1" />
-    </inertial>
-    <visual>
-      <origin
-        xyz="0 0 0"
-        rpy="0 0 0" />
-      <geometry>
-        <mesh
-          filename="package://timda_body_description/meshes/slide_right.STL" />
-      </geometry>
-      <material
-        name="">
-        <color
-          rgba="0.89804 0.91765 0.92941 1" />
-      </material>
-    </visual>
-    <collision>
-      <origin
-        xyz="0 0 0"
-        rpy="0 0 0" />
-      <geometry>
-        <mesh
-          filename="package://timda_body_description/meshes/slide_right.STL" />
-      </geometry>
-    </collision>
-  </link>
-  <joint
-    name="joint_right"
-    type="prismatic">
-    <origin
-      xyz="-0.2 0.0765 1.1815"
-      rpy="0 0 0" />
-    <parent
-      link="base_link" />
-    <child
-      link="slide_right" />
-    <axis
-      xyz="0 0 1" />
-    <limit
-      lower="-0.8"
-      upper="0"
-      effort="9000"
-      velocity="6.5" />
-    <dynamics damping="7"/>
-  </joint>
-  <link
-    name="slide_left">
-    <inertial>
-      <origin
-        xyz="-1.5722E-05 0.006626 2.4586E-06"
-        rpy="0 0 0" />
-      <mass
-        value="0.24709" />
-      <inertia
-        ixx="1"
-        ixy="0"
-        ixz="0"
-        iyy="1"
-        iyz="0"
-        izz="1" />
-    </inertial>
-    <visual>
-      <origin
-        xyz="0 0 0"
-        rpy="0 0 0" />
-      <geometry>
-        <mesh
-          filename="package://timda_body_description/meshes/slide_right.STL" />
-      </geometry>
-      <material
-        name="">
-        <color
-          rgba="0.89804 0.91765 0.92941 1" />
-      </material>
-    </visual>
-    <collision>
-      <origin
-        xyz="0 0 0"
-        rpy="0 0 0" />
-      <geometry>
-        <mesh
-          filename="package://timda_body_description/meshes/slide_right.STL" />
-      </geometry>
-    </collision>
-  </link>
-  <joint
-    name="joint_left"
-    type="prismatic">
-    <origin
-      xyz="-0.2 -0.0765 1.1815"
-      rpy="0 0 3.1416" />
-    <parent
-      link="base_link" />
-    <child
-      link="slide_left" />
-    <axis
-      xyz="0 0 1" />
-    <limit
-      lower="-0.8"
-      upper="0"
-      effort="9000"
-      velocity="6.5" />
-    <dynamics damping="7"/>
-  </joint>
-  <transmission name="slide_tran_r">
-    <type>transmission_interface/SimpleTransmission</type>
-    <joint name="joint_right">
-      <hardwareInterface>hardware_interface/EffortJointInterface</hardwareInterface>
+        xyz="-0.2 -0.0765 1.1815"
+        rpy="0 0 3.1416" />
+      <parent
+        link="${prefix}base_link" />
+      <child
+        link="${prefix}slide_left" />
+      <axis
+        xyz="0 0 1" />
+      <limit
+        lower="-0.8"
+        upper="0"
+        effort="9000"
+        velocity="6.5" />
+      <dynamics damping="7"/>
     </joint>
-    <actuator name="slide_motor_r">
-      <hardwareInterface>hardware_interface/EffortJointInterface</hardwareInterface>
-      <mechanicalReduction>1</mechanicalReduction>
-    </actuator>
-  </transmission>
-  <transmission name="slide_tran_l">
-    <type>transmission_interface/SimpleTransmission</type>
-    <joint name="joint_left">
-      <hardwareInterface>hardware_interface/EffortJointInterface</hardwareInterface>
-    </joint>
-    <actuator name="slide_motor_l">
-      <hardwareInterface>hardware_interface/EffortJointInterface</hardwareInterface>
-      <mechanicalReduction>1</mechanicalReduction>
-    </actuator>
-  </transmission>
+    <transmission name="slide_tran_r">
+      <type>transmission_interface/SimpleTransmission</type>
+      <joint name="${prefix}joint_right">
+        <hardwareInterface>hardware_interface/EffortJointInterface</hardwareInterface>
+      </joint>
+      <actuator name="slide_motor_r">
+        <hardwareInterface>hardware_interface/EffortJointInterface</hardwareInterface>
+        <mechanicalReduction>1</mechanicalReduction>
+      </actuator>
+    </transmission>
+    <transmission name="slide_tran_l">
+      <type>transmission_interface/SimpleTransmission</type>
+      <joint name="${prefix}joint_left">
+        <hardwareInterface>hardware_interface/EffortJointInterface</hardwareInterface>
+      </joint>
+      <actuator name="slide_motor_l">
+        <hardwareInterface>hardware_interface/EffortJointInterface</hardwareInterface>
+        <mechanicalReduction>1</mechanicalReduction>
+      </actuator>
+    </transmission>
+    <xacro:timda_body_gazebo prefix="${prefix}" />
+  </xacro:macro>
 </robot>

File: timda_description/urdf/timda.urdf.xacro (robot description, xacro)
@@ -13,9 +13,10 @@
       xyz="0.047646 0.0 0.3"
       rpy="0 0 0" />
-    <parent link="mobile_base_link"/>
-    <child link="base_link"/>
+    <parent link="base_link"/><!--mobile-->
+    <child link="body_base_link"/>
   </joint>
-  <xacro:timda_mobile_platform prefix="mobile_"/>
-  <xacro:single_arm side="r"  parent="slide_right">
+  <xacro:timda_mobile_platform prefix=""/>
+  <xacro:timda_body prefix="body_"/>
+  <xacro:single_arm side="r"  parent="body_slide_right">
     <origin xyz="0.0 0.1151 0.0" rpy="1.57 3.1415926 3.1415926" />
   </xacro:single_arm>
@@ -23,5 +24,5 @@
     <origin xyz="0 -0.016 0" rpy="0 0 -1.57" />
   </xacro:suction> -->
-  <xacro:single_arm side="l"  parent="slide_left">
+  <xacro:single_arm side="l"  parent="body_slide_left">
     <origin xyz="0.0 0.1151 0.0" rpy="-1.57 0 0" />
   </xacro:single_arm>

File: timda_description/urdf/timda_sim_odom.urdf.xacro (robot description, xacro)
@@ -13,9 +13,10 @@
       xyz="0.047646 0.0 0.3"
       rpy="0 0 0" />
-    <parent link="mobile_base_link"/>
-    <child link="base_link"/>
+    <parent link="base_link"/> <!--mobile platform-->
+    <child link="body_base_link"/>
   </joint>
-  <xacro:timda_mobile_platform prefix="mobile_"/>
-  <xacro:single_arm side="r"  parent="slide_right">
+  <xacro:timda_mobile_platform prefix=""/>
+  <xacro:timda_body prefix="body_"/>
+  <xacro:single_arm side="r"  parent="body_slide_right">
     <origin xyz="0.0 0.1151 0.0" rpy="1.57 3.1415926 3.1415926" />
   </xacro:single_arm>
@@ -23,5 +24,5 @@
     <origin xyz="0 -0.016 0" rpy="0 0 -1.57" />
   </xacro:suction> -->
-  <xacro:single_arm side="l"  parent="slide_left">
+  <xacro:single_arm side="l"  parent="body_slide_left">
     <origin xyz="0.0 0.1151 0.0" rpy="-1.57 0 0" />
   </xacro:single_arm>
